File: testbench-PCB/usb_interface.kicad_sch (KiCad schematic)
At the start: 12 parts, among them J1 USB_C_Receptacle_USB2.0, U10 CH340C, U9 USBLC6-2SC6

Commit message: Connecter speaker, added JTAG.
Parts:
- added JP1, JP2: SolderJumper_2_Bridged, symbol Jumper:SolderJumper_2_Bridged
Connections:
- net UART0_RXD: now also JP2.2 (B); no longer U10.3 (RXD)
- net UART0_TXD: now also JP1.2 (B); no longer U10.2 (TXD)
- new net: JP2.1 (A), U10.3 (RXD)
- new net: JP1.1 (A), U10.2 (TXD)
Changed lines of the file:
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@@
 (kicad_sch (version 20230121) (generator eeschema)
   (paper "A4")
+  (bus_alias "UART0" (members "UART0_TXD" "UART0_RXD"))
   (junction (at 46.99 106.68) (diameter 0) (color 0 0 0 0)
   )
@@
   (no_connect (at 62.23 96.52))
   (no_connect (at 228.6 81.28))
-  (bus_entry (at 247.65 66.04) (size -2.54 2.54)
-    (stroke (width 0) (type default))
-  )
-  (bus_entry (at 247.65 68.58) (size -2.54 2.54)
+  (bus_entry (at 254 66.04) (size -2.54 2.54)
+    (stroke (width 0) (type default))
+  )
+  (bus_entry (at 254 68.58) (size -2.54 2.54)
     (stroke (width 0) (type default))
   )
@@
     (stroke (width 0) (type default))
   )
-  (bus (pts (xy 247.65 66.04) (xy 247.65 68.58))
+  (wire (pts (xy 228.6 68.58) (xy 232.41 68.58))
+    (stroke (width 0) (type default))
+  )
+  (bus (pts (xy 254 66.04) (xy 254 68.58))
     (stroke (width 0) (type default))
   )
@@
     (stroke (width 0) (type default))
   )
-  (wire (pts (xy 228.6 68.58) (xy 245.11 68.58))
-    (stroke (width 0) (type default))
-  )
   (wire (pts (xy 151.13 52.07) (xy 151.13 62.23))
     (stroke (width 0) (type default))
@@
     (stroke (width 0) (type default))
   )
+  (wire (pts (xy 240.03 68.58) (xy 251.46 68.58))
+    (stroke (width 0) (type default))
+  )
+  (wire (pts (xy 228.6 71.12) (xy 232.41 71.12))
+    (stroke (width 0) (type default))
+  )
+  (wire (pts (xy 240.03 71.12) (xy 251.46 71.12))
+    (stroke (width 0) (type default))
+  )
   (wire (pts (xy 66.04 86.36) (xy 62.23 86.36))
     (stroke (width 0) (type default))
@@
     (stroke (width 0) (type default))
   )
-  (bus (pts (xy 247.65 66.04) (xy 247.65 52.07))
+  (bus (pts (xy 254 66.04) (xy 254 52.07))
     (stroke (width 0) (type default))
   )
@@
     (stroke (width 0) (type default))
   )
-  (bus (pts (xy 247.65 52.07) (xy 256.54 52.07))
+  (bus (pts (xy 254 52.07) (xy 262.89 52.07))
     (stroke (width 0) (type default))
   )
@@
   )
   (wire (pts (xy 218.44 46.99) (xy 218.44 50.8))
-    (stroke (width 0) (type default))
-  )
-  (wire (pts (xy 228.6 71.12) (xy 245.11 71.12))
     (stroke (width 0) (type default))
   )
@@
     (effects (font (size 2.5 2.5) (thickness 0.254) bold (color 255 0 0 1)) (justify left bottom))
   )
-  (label "UART0_TXD" (at 234.95 68.58 0) (fields_autoplaced)
+  (label "UART0_TXD" (at 241.3 68.58 0) (fields_autoplaced)
     (effects (font (size 1.27 1.27)) (justify left bottom))
   )
-  (label "UART0_RXD" (at 234.95 71.12 0) (fields_autoplaced)
+  (label "UART0_RXD" (at 241.3 71.12 0) (fields_autoplaced)
     (effects (font (size 1.27 1.27)) (justify left bottom))
   )
-  (hierarchical_label "{UART0}" (shape bidirectional) (at 256.54 52.07 0) (fields_autoplaced)
+  (hierarchical_label "{UART0}" (shape bidirectional) (at 262.89 52.07 0) (fields_autoplaced)
     (effects (font (size 1.27 1.27)) (justify left))
   )
@@
         (path "/3ac6901d-218d-4b34-8c4a-bf7c417c33bc/85a3a829-d3a3-466d-ad77-bb3f90e9de82"
           (reference "C9") (unit 1)
+        )
+      )
+    )
+  )
+  (symbol (lib_id "Jumper:SolderJumper_2_Bridged") (at 236.22 71.12 0) (unit 1)
+    (in_bom yes) (on_board yes) (dnp no)
+    (property "Reference" "JP2" (at 236.22 73.66 0)
+      (effects (font (size 1.27 1.27)))
+    )
+    (property "Value" "SolderJumper_2_Bridged" (at 236.22 67.31 0)
+      (effects (font (size 1.27 1.27)) hide)
+    )
+    (property "Footprint" "" (at 236.22 71.12 0)
+      (effects (font (size 1.27 1.27)) hide)
+    )
+    (property "Datasheet" "~" (at 236.22 71.12 0)
+      (effects (font (size 1.27 1.27)) hide)
+    )
+    (pin "1")
+    (pin "2")
+    (instances
+      (project "testbench"
+        (path "/3ac6901d-218d-4b34-8c4a-bf7c417c33bc/85a3a829-d3a3-466d-ad77-bb3f90e9de82"
+          (reference "JP2") (unit 1)
         )
       )
@@
     )
   )
+  (symbol (lib_id "Jumper:SolderJumper_2_Bridged") (at 236.22 68.58 0) (unit 1)
+    (in_bom yes) (on_board yes) (dnp no)
+    (property "Reference" "JP1" (at 236.22 66.04 0)
+      (effects (font (size 1.27 1.27)))
+    )
+    (property "Value" "SolderJumper_2_Bridged" (at 236.22 64.77 0)
+      (effects (font (size 1.27 1.27)) hide)
+    )
+    (property "Footprint" "" (at 236.22 68.58 0)
+      (effects (font (size 1.27 1.27)) hide)
+    )
+    (property "Datasheet" "~" (at 236.22 68.58 0)
+      (effects (font (size 1.27 1.27)) hide)
+    )
+    (pin "1")
+    (pin "2")
+    (instances
+      (project "testbench"
+        (path "/3ac6901d-218d-4b34-8c4a-bf7c417c33bc/85a3a829-d3a3-466d-ad77-bb3f90e9de82"
+          (reference "JP1") (unit 1)
+        )
+      )
+    )
+  )
   (symbol (lib_id "Device:Polyfuse") (at 99.06 57.15 90) (unit 1)
     (in_bom yes) (on_board yes) (dnp no) (fields_autoplaced)
@@
   )
   (symbol (lib_id "Device:FerriteBead") (at 39.37 110.49 0) (unit 1)
-    (in_bom yes) (on_board yes) (dnp no) (fields_autoplaced)
-    (property "Reference" "FB1" (at 43.18 109.1692 0)
-      (effects (font (size 1.27 1.27)) (justify left))
-    )
-    (property "Value" "100R@100MHz" (at 43.18 111.7092 0)
-      (effects (font (size 1.27 1.27)) (justify left))
-    )
+    (in_bom yes) (on_board yes) (dnp no)
+    (property "Reference" "FB1" (at 31.75 109.22 0)
+      (effects (font (size 1.27 1.27)) (justify left))
+    )
+    (property "Value" "100R@100MHz" (at 21.59 111.76 0)
+      (effects (font (size 1.27 1.27)) (justify left))
+    )

Commit message: Created PCB, changed footprints for symbols.
Parts:
- J1: footprint (none) -> Connector_USB:USB_C_Receptacle_HRO_TYPE-C-31-M-12
- JP1, JP2: footprint (none) -> Jumper:SolderJumper-2_P1.3mm_Bridged2Bar_RoundedPad1.0x1.5mm
Changed lines of the file:
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@@
       (effects (font (size 1.27 1.27)) hide)
     )
-    (property "Footprint" "" (at 236.22 71.12 0)
+    (property "Footprint" "Jumper:SolderJumper-2_P1.3mm_Bridged2Bar_RoundedPad1.0x1.5mm" (at 236.22 71.12 0)
       (effects (font (size 1.27 1.27)) hide)
     )
@@
       (effects (font (size 1.27 1.27)))
     )
-    (property "Footprint" "" (at 50.8 81.28 0)
+    (property "Footprint" "Connector_USB:USB_C_Receptacle_HRO_TYPE-C-31-M-12" (at 50.8 81.28 0)
       (effects (font (size 1.27 1.27)) hide)
     )
@@
       (effects (font (size 1.27 1.27)) hide)
     )
-    (property "Footprint" "" (at 236.22 68.58 0)
-      (effects (font (size 1.27 1.27)) hide)
-    )
+    (property "Footprint" "Jumper:SolderJumper-2_P1.3mm_Bridged2Bar_RoundedPad1.0x1.5mm" (at 236.22 68.58 0)
+      (effects (font (size 1.27 1.27)) hide)
+    )

Commit message: Routed osc., USB interface.
Parts:
- C1: footprint (none) -> Capacitor_SMD:C_0805_2012Metric
- F1: footprint (none) -> Fuse:Fuse_1812_4532Metric
Connections:
- net VBUS: now reaches F1.1, J1.A4 (VBUS), J1.A9 (VBUS), J1.B4 (VBUS), J1.B9 (VBUS)
Other:
- note removed: "note: make D+ D- parallel in PCB"
Changed lines of the file:
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@@
     (stroke (width 0) (type default))
-  )
-  (text "note: make D+ D- parallel in PCB" (at 118.11 36.83 0)
-    (effects (font (size 2.5 2.5) (thickness 0.254) bold (color 255 0 0 1)) (justify left bottom))
   )
   (label "UART0_TXD" (at 241.3 68.58 0) (fields_autoplaced)
@@
   )
   (label "UART0_RXD" (at 241.3 71.12 0) (fields_autoplaced)
+    (effects (font (size 1.27 1.27)) (justify left bottom))
+  )
+  (label "VBUS" (at 76.2 66.04 0) (fields_autoplaced)
     (effects (font (size 1.27 1.27)) (justify left bottom))
   )
@@
       (effects (font (size 1.27 1.27)) (justify left))
     )
-    (property "Footprint" "" (at 112.7252 66.04 0)
+    (property "Footprint" "Capacitor_SMD:C_0805_2012Metric" (at 112.7252 66.04 0)
       (effects (font (size 1.27 1.27)) hide)
     )
@@
       (effects (font (size 1.27 1.27)))
     )
-    (property "Footprint" "" (at 104.14 55.88 0)
+    (property "Footprint" "Fuse:Fuse_1812_4532Metric" (at 104.14 55.88 0)
       (effects (font (size 1.27 1.27)) (justify left) hide)
     )
