File: testbench-PCB/atmega328p.kicad_sch (KiCad schematic)
At the start: 13 parts, among them U5 ATmega328P_Xplained_Mini

Commit message: Fixed footprints in schematics.
Parts:
- R17, R18, R19, R20, R21, R22, R23, R24, R25, R26, R27, R28: footprint (none) -> Resistor_SMD:R_0805_2012Metric
- U5: value ATmega328P_Xplained_Mini -> ~; footprint kit_modules:ATmega328P_Xplained_Mini -> kit_modules:ATmega328P_Xplained_mini

Commit message: Routing the PCB.
Connections:
- net DUT_D7: now reaches U5.1 (PD0)
- net DUT_D16: now reaches U5.10 (PB1)
- net DUT_D17: now reaches U5.11 (PB2)
- net DUT_D8: now reaches U5.2 (PD1)
- net DUT_D9: now reaches U5.3 (PD2)
- net DUT_D10: now reaches U5.4 (PD3)
- net DUT_D11: now reaches U5.5 (PD4)
- net DUT_D12: now reaches U5.6 (PD5)
- net DUT_D13: now reaches U5.7 (PD6)
- net DUT_D14: now reaches U5.8 (PD7)
- net DUT_D15: now reaches U5.9 (PB0)
- net MISO renamed DUT_D19
- net MOSI renamed DUT_D18
- net SCK renamed DUT_D20
Changed lines of the file:
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@@
-    (stroke (width 0) (type default))
-  )
-  (wire (pts (xy 208.28 91.44) (xy 228.6 91.44))
     (stroke (width 0) (type default))
   )
@@
   )
   (wire (pts (xy 208.28 71.12) (xy 228.6 71.12))
+    (stroke (width 0) (type default))
+  )
+  (wire (pts (xy 208.28 91.44) (xy 228.6 91.44))
     (stroke (width 0) (type default))
   )
@@
     (stroke (width 0) (type default))
   )
-  (wire (pts (xy 208.28 73.66) (xy 228.6 73.66))
-    (stroke (width 0) (type default))
-  )
   (wire (pts (xy 29.21 52.07) (xy 88.9 52.07))
     (stroke (width 0) (type default))
@@
   )
   (wire (pts (xy 39.37 85.09) (xy 29.21 85.09))
+    (stroke (width 0) (type default))
+  )
+  (wire (pts (xy 208.28 73.66) (xy 228.6 73.66))
     (stroke (width 0) (type default))
   )
@@
     (stroke (width 0) (type default))
   )
+  (label "DUT_D11" (at 219.71 86.36 0) (fields_autoplaced)
+    (effects (font (size 1.27 1.27)) (justify left bottom))
+  )
+  (label "DUT_D8" (at 219.71 93.98 0) (fields_autoplaced)
+    (effects (font (size 1.27 1.27)) (justify left bottom))
+  )
   (label "DUT_D4" (at 137.16 90.17 0) (fields_autoplaced)
     (effects (font (size 1.27 1.27)) (justify left bottom))
-  )
-  (label "SCK" (at 228.6 60.96 180) (fields_autoplaced)
-    (effects (font (size 1.27 1.27)) (justify right bottom))
   )
   (label "DUT_D6" (at 137.16 95.25 0) (fields_autoplaced)
@@
     (effects (font (size 1.27 1.27)) (justify left bottom))
   )
-  (label "MISO" (at 228.6 63.5 180) (fields_autoplaced)
-    (effects (font (size 1.27 1.27)) (justify right bottom))
+  (label "DUT_D14" (at 219.71 78.74 0) (fields_autoplaced)
+    (effects (font (size 1.27 1.27)) (justify left bottom))
   )
-  (label "MOSI" (at 228.6 66.04 180) (fields_autoplaced)
-    (effects (font (size 1.27 1.27)) (justify right bottom))
+  (label "DUT_D17" (at 219.71 68.58 0) (fields_autoplaced)
+    (effects (font (size 1.27 1.27)) (justify left bottom))
   )
   (label "DUT_D1" (at 82.55 52.07 0) (fields_autoplaced)
@@
     (effects (font (size 1.27 1.27)) (justify left bottom))
   )
+  (label "DUT_D19" (at 219.71 63.5 0) (fields_autoplaced)
+    (effects (font (size 1.27 1.27)) (justify left bottom))
+  )
   (label "DUT_D2" (at 137.16 85.09 0) (fields_autoplaced)
+    (effects (font (size 1.27 1.27)) (justify left bottom))
+  )
+  (label "DUT_D7" (at 219.71 96.52 0) (fields_autoplaced)
+    (effects (font (size 1.27 1.27)) (justify left bottom))
+  )
+  (label "DUT_D12" (at 219.71 83.82 0) (fields_autoplaced)
+    (effects (font (size 1.27 1.27)) (justify left bottom))
+  )
+  (label "DUT_D10" (at 219.71 88.9 0) (fields_autoplaced)
     (effects (font (size 1.27 1.27)) (justify left bottom))
   )
@@
     (effects (font (size 1.27 1.27)) (justify left bottom))
   )
+  (label "DUT_D18" (at 219.71 66.04 0) (fields_autoplaced)
+    (effects (font (size 1.27 1.27)) (justify left bottom))
+  )
   (label "DUT_D3" (at 82.55 59.69 0) (fields_autoplaced)
     (effects (font (size 1.27 1.27)) (justify left bottom))
   )
+  (label "DUT_D16" (at 219.71 71.12 0) (fields_autoplaced)
+    (effects (font (size 1.27 1.27)) (justify left bottom))
+  )
   (label "DUT_D4" (at 82.55 63.5 0) (fields_autoplaced)
+    (effects (font (size 1.27 1.27)) (justify left bottom))
+  )
+  (label "DUT_D13" (at 219.71 81.28 0) (fields_autoplaced)
+    (effects (font (size 1.27 1.27)) (justify left bottom))
+  )
+  (label "DUT_D20" (at 219.71 60.96 0) (fields_autoplaced)
     (effects (font (size 1.27 1.27)) (justify left bottom))
   )
@@
     (effects (font (size 1.27 1.27)) (justify left bottom))
   )
+  (label "DUT_D15" (at 219.71 73.66 0) (fields_autoplaced)
+    (effects (font (size 1.27 1.27)) (justify left bottom))
+  )
   (label "DUT_D2" (at 82.55 55.88 0) (fields_autoplaced)
     (effects (font (size 1.27 1.27)) (justify left bottom))
   )
+  (label "DUT_D9" (at 219.71 91.44 0) (fields_autoplaced)
+    (effects (font (size 1.27 1.27)) (justify left bottom))
+  )

Commit message: Added protective resistors.
Parts:
- added R14 (x21): 330R, Resistor_SMD:R_0805_2012Metric, symbol Device:R
Connections:
- net DUT_D0: now also R14.1; no longer U5.21 (~{RESET}/PC6)
- net DUT_D1: now also R14.1; no longer R17.2, R18.1, U5.27 (PC0)
- net DUT_D10: now also R14.2; no longer U5.4 (PD3)
- net DUT_D11: now also R14.2; no longer U5.5 (PD4)
- net DUT_D12: now also R14.2; no longer U5.6 (PD5)
- net DUT_D13: now also R14.2; no longer U5.7 (PD6)
- net DUT_D14: now also R14.2; no longer U5.8 (PD7)
- net DUT_D15: now also R14.2; no longer U5.9 (PB0)
- net DUT_D16: now also R14.2; no longer U5.10 (PB1)
- net DUT_D17: now also R14.2; no longer U5.11 (PB2)
- net DUT_D18: now also R14.2; no longer U5.12 (PB3)
- net DUT_D19: now also R14.2; no longer U5.13 (PB4)
- net DUT_D2: now also R14.1; no longer R19.2, R20.1, U5.28 (PC1)
- net DUT_D20: now also R14.2; no longer U5.14 (PB5)
- net DUT_D3: now also R14.1; no longer R21.2, R22.1, U5.29 (PC2)
- net DUT_D4: now also R14.1; no longer R23.2, R24.1, U5.30 (PC3)
- net DUT_D5: now also R14.1; no longer R25.2, R26.1, U5.31 (PC4)
- net DUT_D6: now also R14.1; no longer R27.2, R28.1, U5.32 (PC5)
- net DUT_D7: now also R14.2; no longer U5.1 (PD0)
- net DUT_D8: now also R14.2; no longer U5.2 (PD1)
- net DUT_D9: now also R14.2; no longer U5.3 (PD2)
- new net D0: R14.2, U5.21 (~{RESET}/PC6)
- new net D1: R14.2, R17.2, R18.1, U5.27 (PC0)
- new net D10: R14.1, U5.11 (PB2)
- new net D11: R14.1, U5.10 (PB1)
- new net D12: R14.1, U5.9 (PB0)
- new net D13: R14.1, U5.8 (PD7)
- new net D14: R14.1, U5.7 (PD6)
- new net D15: R14.1, U5.6 (PD5)
- new net D16: R14.1, U5.5 (PD4)
- new net D17: R14.1, U5.4 (PD3)
- new net D18: R14.1, U5.3 (PD2)
- new net D19: R14.1, U5.2 (PD1)
- new net D2: R14.2, R19.2, R20.1, U5.28 (PC1)
- new net D20: R14.1, U5.1 (PD0)
- new net D3: R14.2, R21.2, R22.1, U5.29 (PC2)
- new net D4: R14.2, R23.2, R24.1, U5.30 (PC3)
- new net D5: R14.2, R25.2, R26.1, U5.31 (PC4)
- new net D6: R14.2, R27.2, R28.1, U5.32 (PC5)
- new net D7: R14.1, U5.14 (PB5)
- new net D8: R14.1, U5.13 (PB4)
- new net D9: R14.1, U5.12 (PB3)
Other:
- moved on the sheet: R17, R18, R19, R20, R21, R22, R23, R24, R25, R26, R27, R28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
