File: testbench-PCB/atmega328p.kicad_sch (KiCad schematic)
At the start: 34 parts

Commit message: Added titles to schematics.
Other:
- note added: "ATmega328P module"
- company: (none) -> Company: VUT Brno
- title: (none) -> Test benches for microcontroller kits
Changed lines of the file:
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@@
 (kicad_sch (version 20230121) (generator eeschema)
   (paper "A4")
+  (title_block
+    (title "Test benches for microcontroller kits")
+    (date "2023")
+    (rev "v0.1")
+    (company "Company: VUT Brno")
+    (comment 1 "Author: Ivo Zaludek")
+  )
   (junction (at 64.77 172.72) (diameter 0) (color 0 0 0 0)
   )
@@
     (stroke (width 0) (type default))
   )
+  (text "ATmega328P module" (at 177.8 173.99 0)
+    (effects (font (size 5 5)) (justify left bottom))
+  )
   (label "D16" (at 168.91 86.36 0) (fields_autoplaced)
